File: sechs-oszilleieren/sechs-oszilleiren/sechs-oszilleiren_backup.sch (KiCad schematic (older format))
At the start: 53 parts, among them J107 AudioJack2, J108 AudioJack2, J109 AudioJack2, J110 Conn_IDC_Box_Header_02x05_Top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, Q104 2N3904, Q105 2N3904, U101 40106, U102 TL072

Commit message: Added board connector pins and reformatted the schematic to account for 2 board design.
Parts:
- removed C1, C111, C114: 0.1uF, Capacitor_SMD:C_0805_2012Metric, symbol Device:C_Small
- removed C101, C102, C103: 1.0uF, Capacitor_SMD:C_0805_2012Metric, symbol Device:C
- removed C104, C105, C106: 0.1uF, Capacitor_SMD:C_0805_2012Metric, symbol Device:C
- removed C107: 0.01uF, Capacitor_SMD:C_0805_2012Metric, symbol Device:C_Small
- removed C108, C112, C113, C? (x2): 10uF, Capacitor_SMD:CP_Elec_5x5.4, symbol Device:CP1_Small
- removed C109: 47pF, Capacitor_SMD:C_0805_2012Metric, symbol Device:C_Small
- removed C110: 27pF, Capacitor_SMD:C_0805_2012Metric, symbol Device:C_Small
- removed D104, D105, D106: 1N4148, Diode_SMD:D_SOD-323, symbol Device:D_Small_ALT
- removed D107, D108: R, LED_THT:LED_D3.0mm, symbol Device:LED_Small_ALT
- removed J107, J108, J109: AudioJack2, Connector_Audio:Jack_3.5mm_QingPu_WQP-PJ398SM_Vertical_CircularHoles, symbol Connector:AudioJack2
- removed J110: Conn_IDC_Box_Header_02x05_Top_Bottom, Connectors_IDC:IDC-Header_2x05_Pitch2.54mm_Straight, symbol Conn_IDC_Eurorack:Conn_IDC_Box_Header_02x05_Top_Bottom
- removed Q104, Q105: 2N3904, Package_TO_SOT_SMD:SOT-23, symbol Transistor_BJT:2N3904
- removed R107, R108, R109: 1K, Resistor_SMD:R_0805_2012Metric, symbol Device:R_Small_US
- removed R110, R111, R125: 47K, Resistor_SMD:R_0805_2012Metric, symbol Device:R_Small_US
- removed R113, R114: 2K, Resistor_SMD:R_0805_2012Metric, symbol Device:R_Small_US
- removed R116, R117, R118, R119, R120, R121, R122, R123, R124: 10K, Resistor_SMD:R_0805_2012Metric, symbol Device:R_Small_US
- removed R126, R127, R? (x2): 100R, Resistor_SMD:R_0805_2012Metric, symbol Device:R_Small_US
- removed RV107, RV?: A10K, Potentiometer_THT:Potentiometer_Alpha_RD901F-40-00D_Single_Vertical_CircularHoles, symbol Device:R_POT_US
- removed U101: 40106, Package_SO:SOIC-14_3.9x8.7mm_P1.27mm, symbol 4xxx:40106
- removed U102: TL072, Package_SO:SOIC-8_3.9x4.9mm_P1.27mm, symbol Amplifier_Operational:TL072
Connections:
- net labels removed: +12V, GND, MIX_A, MIX_B, MIX_C, MIX_D, MIX_E, MIX_F
- wire segments 177 -> 0
- no-connect marks 2 -> 0
Other:
- note removed: "LEVEL"
- note removed: "LFO Stage"
- note removed: "OUPUT \nMIXER \nSTAGE"
- note removed: "POWER SUPPLY"
- note removed: "VCO Stage"
