File: sechs-oszilleieren/sechs-oszilleiren/output_control_clustersch.sch (KiCad schematic (older format))
At the start: 0 parts

Commit message: Rearranged labeling on voice board, simplified output stage and reduced part count. Simplified CD40106 feedback nets.
Parts:
- added C?: C_Small, symbol 4ms-passives:C_Small
- added RV? (x8): B10K, Potentiometer_THT:Potentiometer_Bourns_PTV09A-1_Single_Vertical, symbol Device:R_POT_US
- added RV? (x6): B100K, Potentiometer_THT:Potentiometer_Bourns_PTV09A-1_Single_Vertical, symbol Device:R_POT_US
Connections:
- new net: RV?.1, RV?.2, RV?.2 (x6)
- new net: C?.2, RV?.3, RV?.3, RV?.3, RV?.3, RV?.3, RV?.3
- new net: C?.1, RV?.1
- new net GAIN_W: RV?.2
- new net GND: RV?.3, RV?.3
- new net LVL_A: RV?.1
- new net LVL_W: RV?.2
- new net SQR_A: RV?.1
- new net SQR_B: RV?.1
- new net SQR_C: RV?.1
- new net SQR_D: RV?.1
- new net SQR_E: RV?.1
- new net SQR_F: RV?.1
- new net TRI_A: RV?.3
- new net TRI_B: RV?.3
- new net TRI_C: RV?.3
- new net TRI_D: RV?.3
- new net TRI_E: RV?.3
- new net TRI_F: RV?.3
