File: sechs-oszilleieren/sechs-oszilleiren/sechs-oszilleiren.kicad_pcb (KiCad board)
At the start: 2 copper layers, 140.2 x 112 mm, 100 parts, among them J1 AudioJack2, J10 AudioJack2, J11 AudioJack2, J12 AudioJack2, J13 AudioJack2, J14 AudioJack2, J15 AudioJack2, J16 Conn_01x02_Male, J17 AudioJack2, J18 AudioJack2, J19 Conn_01x09_Male, J2 AudioJack2, J20 Conn_01x12_Male, J21 Conn_01x06_Male, J22 Conn_01x05_Male, J23 Conn_IDC_Box_Header_02x05_Top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, J24 Conn_01x02_Female, J25 Conn_01x09_Female, J26 Conn_01x12_Female, J27 Conn_01x06_Female, J28 Conn_01x05_Female, J3 AudioJack2, J4 AudioJack2, J5 AudioJack2, J6 AudioJack2, J7 AudioJack2, J8 AudioJack2, J9 AudioJack2, Q1 2N3904, Q2 2N3904, Q3 2N3904, Q4 2N3904, Q5 2N3904, Q6 2N3904, Q7 2N3904, U1 40106, U2 TL072

Commit message: Added a number of stages for the attenuverter, vco, and sechs_oszilleieren.
Parts:
- moved D2 333.3 mm to (10.8, -12.6)
- moved D3 333.3 mm to (-3.38, 1.51)
- moved D4 333.3 mm to (-9.89, 7.54)
- moved D5 333.3 mm to (11.4, -18.4)
- moved D7 333.3 mm to (-19.1, 11.4)
- moved D8 333.3 mm to (-3.38, -4.04)
- moved Q2 333.3 mm to (-9.58, 2.23)
- moved Q6 333.3 mm to (-9.58, -3.56)
- moved D1 333.3 mm to (4.91, -7.09)
- moved D6 333.3 mm to (4.91, -12.6)
- moved Q1 333.3 mm to (-25.3, 17.7)
- moved Q3 333.3 mm to (16.3, -27.6)
- moved Q4 333.3 mm to (-25.3, 11.9)
- moved Q5 333.3 mm to (5.22, -18.0)
- moved Q7 333.3 mm to (16.3, -33.4)
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
Commit message: Rearranged labeling on voice board, simplified output stage and reduced part count. Simplified CD40106 feedback nets.
Parts:
- moved J20 135.8 mm to (-110.0, 63.0)
- moved J16 116.6 mm to (104.0, -12.5)
- moved C1 108.9 mm to (120.0, 88.0)
- moved R1 104.6 mm to (40.5, 13.2)
- moved R10 104.6 mm to (40.5, -7.66)
- moved R11 104.6 mm to (40.5, 7.07)
- moved R12 104.6 mm to (40.5, 5.04)
- moved R13 104.6 mm to (40.4, -5.63)
- moved R15 104.6 mm to (40.5, 0.98)
- moved R4 104.6 mm to (40.4, 15.2)
- moved R5 104.6 mm to (40.5, 11.1)
- moved R6 104.6 mm to (40.4, -1.49)
- moved R7 104.6 mm to (40.5, 9.10)
- moved R8 104.6 mm to (40.4, -3.47)
- moved R9 104.6 mm to (40.5, 17.2)
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Routing:
- removed copper zone on B.Cu, net GND
Other:
- board outline removed
