File: sechs-oszilleieren/sechs-oszilleiren/voice_board.sch (KiCad schematic (older format))
At the start: 42 parts

Commit message: Added board connector pins and reformatted the schematic to account for 2 board design.
Parts:
- removed D?: R, LED_THT:LED_D3.0mm, symbol Device:LED_Small_ALT
- removed R?: 22K, Resistor_SMD:R_0805_2012Metric, symbol Device:R_Small_US
- added C? (x2): 10uF, Capacitor_SMD:CP_Elec_5x5.4, symbol Device:CP1_Small
- added J?: Conn_01x02_Female, symbol Connector:Conn_01x02_Female
- added J?: Conn_01x05_Female, symbol Connector:Conn_01x05_Female
- added J?: Conn_01x06_Female, symbol Connector:Conn_01x06_Female
- added J?: Conn_01x12_Female, symbol Connector:Conn_01x12_Female
- added J?: Conn_01x09_Female, symbol Connector:Conn_01x09_Female
- added R? (x2): 100R, Resistor_SMD:R_0805_2012Metric, symbol Device:R_Small_US
Connections:
- net labels added: level_pot_1, level_pot_w, output_1, output_2, output_indicator, vco_a_cv, vco_a_out, vco_a_pitch_1, vco_a_pitch_3, vco_b_cv, vco_b_out, vco_b_pitch_1, vco_b_pitch_3, vco_c_cv, vco_c_out, vco_c_pitch_1, vco_c_pitch_3, vco_d_cv, vco_d_out, vco_d_pitch_1, vco_d_pitch_3, vco_d_sync, vco_e_cv, vco_e_out, vco_e_pitch_1, vco_e_pitch_3, vco_e_sync, vco_f_cv, vco_f_out, vco_f_pitch_1, vco_f_pitch_3, vco_f_sync
- wire segments 130 -> 264
Other:
- note added: "IC DECOUPLING"
- note added: "LFO STAGE"
- note added: "VCO STAGE"
- moved on the sheet: C?, D?, R?, U?A, U?B, U?C, U?D, U?E, U?F, U?G

Commit message: Added pins between boards for stacking. Changed all components to THT components.
Parts:
- C1, C2, C3: renamed from C?; footprint Capacitor_SMD:C_0805_2012Metric -> Capacitor_THT:C_Rect_L7.2mm_W3.5mm_P5.00mm_FKS2_FKP2_MKS2_MKP2
- C10, C14, C4, C5, C6, C7, C8, C9: renamed from C?; footprint Capacitor_SMD:C_0805_2012Metric -> Capacitor_THT:C_Rect_L7.2mm_W2.5mm_P5.00mm_FKS2_FKP2_MKS2_MKP2
- C11: renamed from C?; footprint Capacitor_SMD:C_0805_2012Metric -> Capacitor_THT:C_Disc_D4.7mm_W2.5mm_P5.00mm
- C12, C13, C15: renamed from C?; footprint Capacitor_SMD:CP_Elec_5x5.4 -> Capacitor_THT:CP_Radial_D5.0mm_P2.50mm
- D10, D11, D9: renamed from D?; footprint Diode_SMD:D_SOD-323 -> Diode_THT:D_DO-35_SOD27_P7.62mm_Horizontal
- J23: renamed from J?; symbol Conn_IDC_Eurorack:Conn_IDC_Box_Header_02x05_Top_Bottom -> sechs-oszilleiren-rescue:Conn_IDC_Box_Header_02x05_Top_Bottom-Conn_IDC_Eurorack
- J24: renamed from J?; footprint (none) -> Connector_PinSocket_2.54mm:PinSocket_1x02_P2.54mm_Vertical
- J25: renamed from J?; footprint (none) -> Connector_PinSocket_2.54mm:PinSocket_1x09_P2.54mm_Vertical
- J26: renamed from J?; footprint (none) -> Connector_PinSocket_2.54mm:PinSocket_1x12_P2.54mm_Vertical
- J27: renamed from J?; footprint (none) -> Connector_PinSocket_2.54mm:PinSocket_1x06_P2.54mm_Vertical
- J28: renamed from J?; footprint (none) -> Connector_PinSocket_2.54mm:PinSocket_1x05_P2.54mm_Vertical
- R16, R17, R18, R19, R20, R21, R22, R23, R24, R25, R26, R27, R28, R29, R30: renamed from R?; footprint Resistor_SMD:R_0805_2012Metric -> Resistor_THT:R_Axial_DIN0204_L3.6mm_D1.6mm_P7.62mm_Horizontal
- U1: renamed from U?; footprint Package_SO:SOIC-14_3.9x8.7mm_P1.27mm -> Package_DIP:DIP-14_W7.62mm_Socket_LongPads
- U2: renamed from U?; footprint Package_SO:SOIC-8_3.9x4.9mm_P1.27mm -> Package_DIP:DIP-8_W7.62mm_Socket_LongPads

Commit message: Rearranged labeling on voice board, simplified output stage and reduced part count. Simplified CD40106 feedback nets.
Parts:
- removed C12, C13: 10uF, Capacitor_THT:CP_Radial_D5.0mm_P2.50mm, symbol Device:CP1_Small
- removed C2, C3: 1.0uF, Capacitor_THT:C_Rect_L7.2mm_W3.5mm_P5.00mm_FKS2_FKP2_MKS2_MKP2, symbol Device:C
- removed C5, C6: 0.1uF, Capacitor_THT:C_Rect_L7.2mm_W2.5mm_P5.00mm_FKS2_FKP2_MKS2_MKP2, symbol Device:C
- removed D10, D11: 1N4148, Diode_THT:D_DO-35_SOD27_P7.62mm_Horizontal, symbol Device:D_Small_ALT
- removed R17, R18: 1K, Resistor_THT:R_Axial_DIN0204_L3.6mm_D1.6mm_P7.62mm_Horizontal, symbol Device:R_Small_US
- removed R19, R20, R21, R22, R23, R24, R26: 10K, Resistor_THT:R_Axial_DIN0204_L3.6mm_D1.6mm_P7.62mm_Horizontal, symbol Device:R_Small_US
- removed R30: 100R, Resistor_THT:R_Axial_DIN0204_L3.6mm_D1.6mm_P7.62mm_Horizontal, symbol Device:R_Small_US
- added C? (x2): 1.0uF, Capacitor_THT:C_Rect_L7.2mm_W3.5mm_P5.00mm_FKS2_FKP2_MKS2_MKP2, symbol Device:C
- added C? (x2): 0.1uF, Capacitor_THT:C_Rect_L7.2mm_W2.5mm_P5.00mm_FKS2_FKP2_MKS2_MKP2, symbol Device:C
- added D? (x6): 1N5819, Diode_THT:D_DO-41_SOD81_P10.16mm_Horizontal, symbol Diode:1N5819
- added D? (x5): 1N4148, Diode_THT:D_DO-35_SOD27_P7.62mm_Horizontal, symbol Device:D_Small_ALT
- added R? (x2): 1K, Resistor_THT:R_Axial_DIN0204_L3.6mm_D1.6mm_P7.62mm_Horizontal, symbol Device:R_Small_US
Connections:
- net labels added: AUDIO_OUT, CVA, CVA_JACK, CVB, CVB_JACK, CVC, CVC_JACK, CVD, CVD_JACK, CVE, CVE_JACK, CVF, CVF_JACK, FBD_IN, FBD_OUT, FBE_IN, FBE_OUT, FBF_IN, FBF_OUT, FREQA_A, FREQA_B, FREQB_A, FREQB_B, FREQC_A, FREQC_B, FREQD_A, FREQD_B, FREQE_A, FREQE_B, FREQF_A, FREQF_B, GAIN_W, LVL_A, LVL_W, MCV, MSYNC, OUT_LED, SAWD_SW1, SAWD_SW2, SAWE_SW1, SAWE_SW2, SAWF_SW1, SAWF_SW2, SQR_A, SQR_B, SQR_C, SQR_D, SQR_E, SQR_F, SYNCD, SYNCD_JACK, SYNCE, SYNCE_JACK, SYNCF, SYNCF_JACK, TRI_A, TRI_B, TRI_C, TRI_D, TRI_E, TRI_F
- net labels removed: MIX_A, MIX_B, MIX_C, MIX_D, MIX_E, MIX_F, level_pot_1, level_pot_w, output_1, output_2, output_indicator, vco_a_cv, vco_a_out, vco_a_pitch_1, vco_a_pitch_3, vco_b_cv, vco_b_out, vco_b_pitch_1, vco_b_pitch_3, vco_c_cv, vco_c_out, vco_c_pitch_1, vco_c_pitch_3, vco_d_cv, vco_d_out, vco_d_pitch_1, vco_d_pitch_3, vco_d_sync, vco_e_cv, vco_e_out, vco_e_pitch_1, vco_e_pitch_3, vco_e_sync, vco_f_cv, vco_f_out, vco_f_pitch_1, vco_f_pitch_3, vco_f_sync
- wire segments 264 -> 273
Other:
- note added: "MEZZANINE CONNECTORS"
- note added: "OUTPUT MIXER"
- note removed: "LFO STAGE"
- note removed: "OUPUT \nMIXER \nSTAGE"
- note removed: "VCO STAGE"
- moved on the sheet: C1, C10, C11, C4, D9, J28, R16, R25, R27, R28, R29, U1A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
