File: active_dual_mult/active_dual_mult_v2_dual_amp_version/active_dual_mult.sch (KiCad schematic (older format))
At the start: 33 parts, among them J1 EURO_HEADER_10pin, J10 B3Out, J11 B4Out, J2 AIn, J3 A1Out, J4 A2Out, J5 A3Out, J6 A4Out, J7 BIn, J8 B1Out, J9 B2Out, U1 TL074, U2 TL074

Commit message: Rewired PCB in version 2 of RAD124 to leverage dual op-amp packages and minimize number of vias for output channels. Changed op amps to OPA2174 SOIC packages to improve unity-gain stability and reduce phase-inversion problems found in TL07X series op amps.
Parts:
- removed U1, U2: TL074, Package_SO:TSSOP-14_4.4x5mm_P0.65mm, symbol Amplifier_Operational:TL074
- added C3, C4, C7, C8: 0.1u, 4ms_Capacitor:C_0805, symbol active_dual_mult-rescue:C_Small-4ms-passives
- added U1, U2, U3, U4: OPA2134, 4ms_Package_SOIC:SOIC-8_5.28x4.9mm_Pitch1.27mm, symbol Amplifier_Operational:OPA2134
- C10: renamed from C2; footprint Capacitor_SMD:CP_Elec_3x5.4 -> 4ms_Capacitor:C_0805
- C9: renamed from C1; footprint Capacitor_SMD:CP_Elec_3x5.4 -> 4ms_Capacitor:C_0805
- renumbered C3 to C1, C4 to C2, D3 to D1, D4 to D2, D1 to D3, D2 to D4, J2 to J1, J1 to J2, R9 to R5, R5 to R6, R6 to R7, R7 to R8, R8 to R9
Connections:
- net AIn: now also U1.3 (+), U1.5 (+), U2.3 (+), U2.5 (+)
- net BIn: now also U3.3 (+), U3.5 (+), U4.3 (+), U4.5 (+)
- net GND: now also C5.1, C6.1, C3.1, C4.1, C7.1, C8.1; no longer C5.2, C6.2
- net VCC: now also C5.2, C3.2, C7.2, U1.8 (V+), U2.8 (V+), U3.8 (V+), U4.8 (V+); no longer C5.1
- net VEE: now also C6.2, C4.2, C8.2, U1.4 (V-), U2.4 (V-), U3.4 (V-), U4.4 (V-); no longer C6.1
- net at R3.2: now also U2.1, U2.2 (-)
- net at R4.2: now also U2.6 (-), U2.7
- net at R9.2: now also U4.6 (-), U4.7
- net at R1.2: now also U1.1, U1.2 (-)
- net at R2.2: now also U1.6 (-), U1.7
- net at R8.2: now also U4.1, U4.2 (-)
- net at R7.2: now also U3.6 (-), U3.7
- net at R6.2: now also U3.1, U3.2 (-)
Other:
- moved on the sheet: C1, C2, D1, D2, R10, R5
