File: roku_x_san_x_go/RokuXSanXGo/roku_san_go.sch (KiCad schematic (older format))
At the start: 73 parts, among them J1 AudioJack2, J2 VCO_CV_IN, J3 LFO_CV_IN, J4 Conn_IDC_Box_Header_02x05_Top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, U1 TL072, U2 40106, U3 40106, U4 NE556, U5 NE556, U6 NE556

Commit message: Added a new revision for RokuXSanXGo
Parts:
- J4: symbol Conn_IDC_Eurorack:Conn_IDC_Box_Header_02x05_Top_Bottom -> roku_san_go-rescue:Conn_IDC_Box_Header_02x05_Top_Bottom-Conn_IDC_Eurorack
Changed lines of the file:
@@
 EESchema Schematic File Version 4
+LIBS:roku_san_go-cache
 EELAYER 29 0
 EELAYER END
@@
 $EndDescr
 $Comp
-L Conn_IDC_Eurorack:Conn_IDC_Box_Header_02x05_Top_Bottom J4
+L roku_san_go-rescue:Conn_IDC_Box_Header_02x05_Top_Bottom-Conn_IDC_Eurorack J4
 U 1 1 5DEE2DD6
 P 14400 8150
